File: PCB/Keyboard.sch (KiCad schematic (older format))
At the start: 33 parts, among them P1 USB_OTG, SW1 RST, X1 ECS-160-10-36Q-ES-TR

Commit message: Restore production files
I discovered that I had overwritten the PCB files by accident. These are restored from an older version.
Parts:
- removed C?: 100n, symbol Device:C_Small
- removed D?: POWER, SMD-DiscreteB:LED-0402-1005, symbol Keyboard-rescue:Led_Small
- removed J?: JTAG, symbol conn:Conn_02x05_Odd_Even
- removed R? (x3): 510, SMD-DiscreteB:R-0402-1005, symbol Device:R_Small
- removed R?: 1M, SMD-DiscreteB:R-0402-1005, symbol Device:R
- removed TP1, TP13, TP14, TP2, TP3, TP4, TP5, TP6: TESTPOINT, Vias_and_Pads:TestPoint_1.0mm, symbol rbv_pcb_extras:TESTPOINT
- removed U?: STM32F103C8Tx, Housings_QFP:LQFP-48_7x7mm_Pitch0.5mm, symbol stm32:STM32F103C8Tx
- added C11: 1µ, SMD-DiscreteB:C-0402-1005, symbol C
- added C5, C6, C7, C9: 100n, SMD-DiscreteB:C-0402-1005, symbol C
- added ISP1: ATMEL_ISP-6P, SMD-Connectors:ISP-PADS_2mm54, symbol ATMEL_ISP-6P
- added R5: 1k, SMD-DiscreteB:R-0402-1005, symbol R_Small
- added U1: ATMEGA32U4-QFN44, SMD-QFN:VQFN-44_ATMEL, symbol ATMEGA32U4-QFN44
- C1, C12, C2, C3, C4: symbol Device:C -> C
- C10, C8: value 20p -> 15p; symbol Device:C -> C
- D1: value PC13 -> STATUS; symbol Keyboard-rescue:Led_Small -> Led_Small
- F1: symbol Keyboard-rescue:F_Small -> F_Small
- KB1: symbol rbv_keyboard:KEYBOARD-PSION-5MX -> KEYBOARD-PSION-5MX; Farnell (none) -> 2520146; Mouser 649-SFV22R-1STE1HLF -> 538-52437-2233
- P1: symbol Keyboard-rescue:USB_OTG-RESCUE-Keyboard -> USB_OTG-RESCUE-Keyboard
- R1, R2, R3, R4: symbol Device:R -> R
- SW1: symbol Keyboard-rescue:SW_PUSH -> SW_PUSH; Farnell (none) -> 2376538; Mouser 688-SKRMAB -> 688-SKRMAA
- X1: value ECS-160-10-36Q-ES-TR -> ABM10-16.000MHZ-D30-T3; symbol rbv_device:CRYSTAL-4pin -> CRYSTAL-4pin; Farnell (none) -> 2467762; Mouser 520-160-10-36Q-EST -> 815-ABM10-16-D30T3
Connections:
- net labels added: MISO, MOSI, SCK, TMP, VARef, VUCap
- net labels removed: +3V3, OSCIN, OSCOUT, PC13, RTCK, TCLK, TDI, TDO, TMS
- wire segments 146 -> 131
- no-connect marks 0 -> 1
Other:
- moved on the sheet: C10, C12, C8, D1, F1, KB1, P1, R1, R2, R3, R4, SW1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
