File: PCB/Keyboard.sch (KiCad schematic (older format))
At the start: 25 parts, among them P1 USB_OTG, SW1 RST, U1 ATMEGA32U4-QFN44, X1 ABM10-16.000MHZ-D30-T3

Commit message: Switched to new library names
At least for the PCB
Parts:
- added J1: RESET, SMD-Connectors:TESTPOINT-1mm-NO_TEXT, symbol conn:TEST_1P
- added J2: SCK, SMD-Connectors:TESTPOINT-1mm-NO_TEXT, symbol conn:TEST_1P
- added J23: 5V, SMD-Connectors:TESTPOINT-1mm-NO_TEXT, symbol conn:TEST_1P
- added J26: GND, SMD-Connectors:TESTPOINT-1mm-NO_TEXT, symbol conn:TEST_1P
- added J3: MISO, SMD-Connectors:TESTPOINT-1mm-NO_TEXT, symbol conn:TEST_1P
- added J4: MOSI, SMD-Connectors:TESTPOINT-1mm-NO_TEXT, symbol conn:TEST_1P
Connections:
- wire segments 164 -> 172
Changed lines of the file:
@@
 	9200 1500 9200 1650
-Wire Wire Line
-	9350 1400 9050 1400
-Wire Wire Line
-	7550 1300 7850 1300
-Wire Wire Line
-	7850 1400 7550 1400
-Wire Wire Line
-	7550 1500 7850 1500
 Wire Wire Line
 	6750 2650 7050 2650
@@
 Wire Wire Line
 	9850 4850 9850 4950
+$Comp
+L conn:TEST_1P J23
+U 1 1 5BA336D5
+P 2700 4300
+F 0 "J23" H 2758 4420 50  0000 L CNN
+F 1 "5V" H 2758 4329 50  0000 L CNN
+F 2 "SMD-Connectors:TESTPOINT-1mm-NO_TEXT" H 2900 4300 50  0001 C CNN
+F 3 "" H 2900 4300 50  0001 C CNN
+	1    2700 4300
+	1    0    0    -1
+$EndComp
+Wire Wire Line
+	2700 4300 2700 4350
+Wire Wire Line
+	2700 4350 2550 4350
+Connection ~ 2550 4350
+$Comp
+L conn:TEST_1P J26
+U 1 1 5BA4EE50
+P 1900 4800
+F 0 "J26" H 1842 4827 50  0000 R CNN
+F 1 "GND" H 1842 4918 50  0000 R CNN
+F 2 "SMD-Connectors:TESTPOINT-1mm-NO_TEXT" H 2100 4800 50  0001 C CNN
+F 3 "" H 2100 4800 50  0001 C CNN
+	1    1900 4800
+	-1   0    0    1
+$EndComp
+Wire Wire Line
+	1650 4750 1900 4750
+Wire Wire Line
+	1900 4750 1900 4800
+Connection ~ 1650 4750
+$Comp
+L conn:TEST_1P J1
+U 1 1 5BA582A5
+P 6650 1000
+F 0 "J1" H 6708 1120 50  0000 L CNN
+F 1 "RESET" H 6708 1029 50  0000 L CNN
+F 2 "SMD-Connectors:TESTPOINT-1mm-NO_TEXT" H 6850 1000 50  0001 C CNN
+F 3 "" H 6850 1000 50  0001 C CNN
+	1    6650 1000
+	1    0    0    -1
+$EndComp
+$Comp
+L conn:TEST_1P J3
+U 1 1 5BA6AA8B
+P 7350 1000
+F 0 "J3" H 7292 1120 50  0000 R CNN
+F 1 "MISO" H 7292 1029 50  0000 R CNN
+F 2 "SMD-Connectors:TESTPOINT-1mm-NO_TEXT" H 7550 1000 50  0001 C CNN
+F 3 "" H 7550 1000 50  0001 C CNN
+	1    7350 1000
+	-1   0    0    -1
+$EndComp
+Wire Wire Line
+	7350 1000 7350 1300
+Wire Wire Line
+	7350 1300 7850 1300
+$Comp
+L conn:TEST_1P J2
+U 1 1 5BA74139
+P 7000 1000
+F 0 "J2" H 7058 1120 50  0000 L CNN
+F 1 "SCK" H 7058 1029 50  0000 L CNN
+F 2 "SMD-Connectors:TESTPOINT-1mm-NO_TEXT" H 7200 1000 50  0001 C CNN
+F 3 "" H 7200 1000 50  0001 C CNN
+	1    7000 1000
+	1    0    0    -1
+$EndComp
+Wire Wire Line
+	7000 1000 7000 1400
+Wire Wire Line
+	7000 1400 7850 1400
+$Comp
+L conn:TEST_1P J4
+U 1 1 5BABDEEC
+P 9450 1000
+F 0 "J4" H 9392 1120 50  0000 R CNN
+F 1 "MOSI" H 9392 1029 50  0000 R CNN
+F 2 "SMD-Connectors:TESTPOINT-1mm-NO_TEXT" H 9650 1000 50  0001 C CNN
+F 3 "" H 9650 1000 50  0001 C CNN
+	1    9450 1000
+	-1   0    0    -1
+$EndComp
+Wire Wire Line
+	9450 1000 9450 1400
+Wire Wire Line
+	9050 1400 9450 1400
+Wire Wire Line
+	6650 1000 6650 1500
+Wire Wire Line
+	6650 1500 7850 1500
 Wire Bus Line
 	7300 2650 7300 5150

Commit message: Added test points
For ICSP and USB. Keyboard connections are tested through a flex cable. LEDs are tested visually.
Parts:
- removed ISP1: ATMEL_ISP-6P, SMD-Connectors:ISP-PADS_2mm54, symbol rbv_mcu:ATMEL_ISP-6P
- added J5: D-, RB-SMD-Connectors:TESTPOINT-1mm-NO_TEXT, symbol conn:TEST_1P
- added J6: D+, RB-SMD-Connectors:TESTPOINT-1mm-NO_TEXT, symbol conn:TEST_1P
- added J7: VBUS, RB-SMD-Connectors:TESTPOINT-1mm-NO_TEXT, symbol conn:TEST_1P
- C1, C10, C11, C12, C2, C3, C4, C5, C6, C7, C8, C9: footprint SMD-DiscreteB:C-0402-1005 -> RB-SMD-DiscreteB:C-0402-1005
- D1: footprint SMD-DiscreteB:LED-0402-1005 -> RB-SMD-DiscreteB:LED-0402-1005
- F1: footprint SMD-DiscreteB:F-0603-1608 -> RB-SMD-DiscreteB:F-0603-1608
- J1, J2, J23, J26, J3, J4: footprint SMD-Connectors:TESTPOINT-1mm-NO_TEXT -> RB-SMD-Connectors:TESTPOINT-1mm-NO_TEXT
- KB1: footprint SMD-Connectors:FPC_0.5mm_22p-MOLEX_52437 -> RB-SMD-Connectors:FPC_0.5mm_22p-MOLEX_52437
- P1: footprint SMD-Connectors:USB-MICRO-10104110-0001LF -> RB-SMD-Connectors:USB-MICRO-10104110-0001LF
- R1, R2, R3, R4, R5: footprint SMD-DiscreteB:R-0402-1005 -> RB-SMD-DiscreteB:R-0402-1005
- SW1: value RST -> RESET; footprint SMD-Switches:ALPS-SKRMAAE010 -> RB-SMD-Switches:ALPS-SKRMAAE010
- U1: footprint SMD-QFN:VQFN-44_ATMEL -> RB-SMD-QFN:VQFN-44_ATMEL
- X1: footprint SMD-XTAL:2.5x2mm -> RB-SMD-XTAL:2.5x2mm
Connections:
- wire segments 172 -> 178
Other:
- note added: "ICSP"
- moved on the sheet: F1, R1, R2

Commit message: Final fixes
Re-annotation, version numbering of schematic
Parts:
- renumbered C8 to C11, C9 to C8, C11 to C9, J7 to J5, J23 to J6, J5 to J7, J6 to J8, J26 to J9, R3 to R1, R1 to R2, R2 to R3
Changed lines of the file:
@@
 encoding utf-8
 Sheet 1 1
-Title ""
-Date ""
-Rev ""
-Comp ""
+Title "USB Keyboard Adapter for Psion 5/5mx"
+Date "2018-09-26"
+Rev "v1.22"
+Comp "Rasmus Backman"
 Comment1 ""
 Comment2 ""
@@
 	7300 5150 7200 5250
 $Comp
-L power:+5V #PWR01
+L power:+5V #PWR03
 U 1 1 54DFCCB0
 P 5150 1400
-F 0 "#PWR01" H 5150 1250 60  0001 C CNN
+F 0 "#PWR03" H 5150 1250 60  0001 C CNN
 F 1 "+5V" H 5150 1540 60  0000 C CNN
 F 2 "" H 5150 1400 60  0000 C CNN
@@
 $EndComp
 $Comp
-L power:GND #PWR02
+L power:GND #PWR018
 U 1 1 54DFCF30
 P 5400 6150
-F 0 "#PWR02" H 5400 5900 60  0001 C CNN
+F 0 "#PWR018" H 5400 5900 60  0001 C CNN
 F 1 "GND" H 5400 6000 60  0000 C CNN
 F 2 "" H 5400 6150 60  0000 C CNN
@@
 $EndComp
 $Comp
-L power:+5V #PWR03
+L power:+5V #PWR04
 U 1 1 54DFC139
 P 5550 1400
-F 0 "#PWR03" H 5550 1250 60  0001 C CNN
+F 0 "#PWR04" H 5550 1250 60  0001 C CNN
 F 1 "+5V" H 5550 1540 60  0000 C CNN
 F 2 "" H 5550 1400 60  0000 C CNN
@@
 $EndComp
 $Comp
-L power:+5V #PWR04
+L power:+5V #PWR05
 U 1 1 54DFC147
 P 5850 1400
-F 0 "#PWR04" H 5850 1250 60  0001 C CNN
+F 0 "#PWR05" H 5850 1250 60  0001 C CNN
 F 1 "+5V" H 5850 1540 60  0000 C CNN
 F 2 "" H 5850 1400 60  0000 C CNN
@@
 $EndComp
 $Comp
-L power:+5V #PWR05
+L power:+5V #PWR01
 U 1 1 54DFC155
 P 850 950
-F 0 "#PWR05" H 850 800 60  0001 C CNN
+F 0 "#PWR01" H 850 800 60  0001 C CNN
 F 1 "+5V" H 850 1090 60  0000 C CNN
 F 2 "" H 850 950 60  0000 C CNN
@@
 $EndComp
 $Comp
-L power:GND #PWR06
+L power:GND #PWR07
 U 1 1 54DFC193
 P 850 1850
-F 0 "#PWR06" H 850 1600 60  0001 C CNN
+F 0 "#PWR07" H 850 1600 60  0001 C CNN
 F 1 "GND" H 850 1700 60  0000 C CNN
 F 2 "" H 850 1850 60  0000 C CNN
@@
 $EndComp
 $Comp
-L Device:C C9
+L Device:C C8
 U 1 1 54DFC828
 P 3650 1400
-F 0 "C9" H 3700 1500 50  0000 L CNN
+F 0 "C8" H 3700 1500 50  0000 L CNN
 F 1 "100n" H 3700 1300 50  0000 L CNN
 F 2 "RB-SMD-DiscreteB:C-0402-1005" H 3688 1250 30  0001 C CNN
@@
 $EndComp
 $Comp
-L Device:C C11
+L Device:C C9
 U 1 1 54DFC82E
 P 4050 1400
-F 0 "C11" H 4100 1500 50  0000 L CNN
+F 0 "C9" H 4100 1500 50  0000 L CNN
 F 1 "1µ" H 4100 1300 50  0000 L CNN
 F 2 "RB-SMD-DiscreteB:C-0402-1005" H 4088 1250 30  0001 C CNN
@@
 VARef
 $Comp
-L power:GND #PWR07
+L power:GND #PWR017
 U 1 1 54DFD489
 P 1650 5700
-F 0 "#PWR07" H 1650 5450 60  0001 C CNN
+F 0 "#PWR017" H 1650 5450 60  0001 C CNN
 F 1 "GND" H 1650 5550 60  0000 C CNN
 F 2 "" H 1650 5700 60  0000 C CNN
@@
 $EndComp
 $Comp
-L Device:C C8
+L Device:C C11
 U 1 1 54DFDE8F
 P 3600 4100
-F 0 "C8" V 3700 4200 50  0000 L CNN
+F 0 "C11" V 3700 4200 50  0000 L CNN
 F 1 "15p" V 3700 4000 50  0000 R CNN
 F 2 "RB-SMD-DiscreteB:C-0402-1005" H 3638 3950 30  0001 C CNN
@@
 $EndComp
 $Comp
-L power:GND #PWR08
+L power:GND #PWR011
 U 1 1 54DFE17B
 P 4400 3800
-F 0 "#PWR08" H 4400 3550 60  0001 C CNN
+F 0 "#PWR011" H 4400 3550 60  0001 C CNN
 F 1 "GND" H 4400 3650 60  0000 C CNN
 F 2 "" H 4400 3800 60  0000 C CNN
@@
 $EndComp
 $Comp
-L power:GND #PWR09
+L power:GND #PWR010
 U 1 1 54DFE3E2
 P 3300 3800
-F 0 "#PWR09" H 3300 3550 60  0001 C CNN
+F 0 "#PWR010" H 3300 3550 60  0001 C CNN
 F 1 "GND" H 3300 3650 60  0000 C CNN
 F 2 "" H 3300 3800 60  0000 C CNN
@@
 $EndComp
 $Comp
-L Device:R R1
+L Device:R R2
 U 1 1 54DFF0F0
 P 2950 4450
-F 0 "R1" V 3030 4450 50  0000 C CNN
+F 0 "R2" V 3030 4450 50  0000 C CNN
 F 1 "22" V 2950 4450 50  0000 C CNN
 F 2 "RB-SMD-DiscreteB:R-0402-1005" V 2880 4450 30  0001 C CNN
@@
 $EndComp
 $Comp
-L Device:R R2
+L Device:R R3
 U 1 1 54DFF139
 P 2950 4550
-F 0 "R2" V 3030 4550 50  0000 C CNN
+F 0 "R3" V 3030 4550 50  0000 C CNN
 F 1 "22" V 2950 4550 50  0000 C CNN
 F 2 "RB-SMD-DiscreteB:R-0402-1005" V 2880 4550 30  0001 C CNN
@@
 $EndComp
 $Comp
-L power:+5V #PWR010
+L power:+5V #PWR013
 U 1 1 54DFF76F
 P 2550 4200
-F 0 "#PWR010" H 2550 4050 60  0001 C CNN
+F 0 "#PWR013" H 2550 4050 60  0001 C CNN
 F 1 "+5V" H 2550 4340 60  0000 C CNN
 F 2 "" H 2550 4200 60  0000 C CNN
@@
 $EndComp
 $Comp
-L Device:R R3
+L Device:R R1
 U 1 1 54E0052B
 P 4450 2500
-F 0 "R3" V 4530 2500 50  0000 C CNN
+F 0 "R1" V 4530 2500 50  0000 C CNN
 F 1 "10k" V 4457 2501 50  0000 C CNN
 F 2 "RB-SMD-DiscreteB:R-0402-1005" V 4380 2500 30  0001 C CNN
@@
 $EndComp
 $Comp
-L power:+5V #PWR011
+L power:+5V #PWR08
 U 1 1 54E0055F
 P 4450 2250
-F 0 "#PWR011" H 4450 2100 60  0001 C CNN
+F 0 "#PWR08" H 4450 2100 60  0001 C CNN
 F 1 "+5V" H 4450 2390 60  0000 C CNN
 F 2 "" H 4450 2250 60  0000 C CNN
@@
 RESET
 $Comp
-L power:+5V #PWR012
+L power:+5V #PWR02
 U 1 1 54E02417
 P 9200 1000
-F 0 "#PWR012" H 9200 850 60  0001 C CNN
+F 0 "#PWR02" H 9200 850 60  0001 C CNN
 F 1 "+5V" H 9200 1140 60  0000 C CNN
 F 2 "" H 9200 1000 60  0000 C CNN
@@
 MOSI
 $Comp
-L power:GND #PWR013
+L power:GND #PWR06
 U 1 1 54E025DE
 P 9200 1650
-F 0 "#PWR013" H 9200 1400 60  0001 C CNN
+F 0 "#PWR06" H 9200 1400 60  0001 C CNN
 F 1 "GND" H 9200 1500 60  0000 C CNN
 F 2 "" H 9200 1650 60  0000 C CNN
@@
 Connection ~ 1650 5400
 $Comp
-L Keyboard-rescue:GNDPWR #PWR014
+L Keyboard-rescue:GNDPWR #PWR016
 U 1 1 5736425E
 P 1050 5700
-F 0 "#PWR014" H 1050 5500 50  0001 C CNN
+F 0 "#PWR016" H 1050 5500 50  0001 C CNN
 F 1 "GNDPWR" H 1050 5570 50  0000 C CNN
 F 2 "" H 1050 5650 50  0000 C CNN
@@
 	3250 2750 3250 2850
 $Comp
-L power:GND #PWR016
+L power:GND #PWR09
 U 1 1 57F3F6A7
 P 3250 2850
-F 0 "#PWR016" H 3250 2600 60  0001 C CNN
+F 0 "#PWR09" H 3250 2600 60  0001 C CNN
 F 1 "GND" H 3250 2700 60  0000 C CNN
 F 2 "" H 3250 2850 60  0000 C CNN
@@
 	9850 4750 9850 4850
 $Comp
-L power:GND #PWR017
+L power:GND #PWR014
 U 1 1 57FBF30B
 P 9850 4950
-F 0 "#PWR017" H 9850 4700 50  0001 C CNN
+F 0 "#PWR014" H 9850 4700 50  0001 C CNN
 F 1 "GND" H 9850 4800 50  0000 C CNN
 F 2 "" H 9850 4950 50  0000 C CNN
@@
 Connection ~ 9850 4850
 $Comp
-L rbv_power:VBUS #PWR018
+L rbv_power:VBUS #PWR012
 U 1 1 583354E1
 P 1800 4200
-F 0 "#PWR018" H 1800 4050 50  0001 C CNN
+F 0 "#PWR012" H 1800 4050 50  0001 C CNN
 F 1 "VBUS" H 1815 4373 50  0000 C CNN
 F 2 "" H 1800 4200 60  0000 C CNN
@@
 	9850 4850 9850 4950
 $Comp
-L conn:TEST_1P J23
+L conn:TEST_1P J6
 U 1 1 5BA336D5
 P 2700 4250
-F 0 "J23" H 2758 4370 50  0000 L CNN
+F 0 "J6" H 2758 4370 50  0000 L CNN
 F 1 "5V" H 2758 4279 50  0000 L CNN
 F 2 "RB-SMD-Connectors:TESTPOINT-1mm-NO_TEXT" H 2900 4250 50  0001 C CNN
@@
 Connection ~ 2550 4350
 $Comp
-L conn:TEST_1P J26
+L conn:TEST_1P J9
 U 1 1 5BA4EE50
 P 1900 4800
-F 0 "J26" H 1842 4827 50  0000 R CNN
+F 0 "J9" H 1842 4827 50  0000 R CNN
 F 1 "GND" H 1842 4918 50  0000 R CNN
 F 2 "RB-SMD-Connectors:TESTPOINT-1mm-NO_TEXT" H 2100 4800 50  0001 C CNN
@@
 ICSP
 $Comp
-L conn:TEST_1P J6
+L conn:TEST_1P J8
 U 1 1 5BAC5EE6
 P 3250 4700
-F 0 "J6" H 3308 4820 50  0000 L CNN
+F 0 "J8" H 3308 4820 50  0000 L CNN
 F 1 "D+" H 3308 4729 50  0000 L CNN
 F 2 "RB-SMD-Connectors:TESTPOINT-1mm-NO_TEXT" H 3450 4700 50  0001 C CNN
@@
 $EndComp
 $Comp
-L conn:TEST_1P J5
+L conn:TEST_1P J7
 U 1 1 5BAC5EEC
 P 3250 4300
-F 0 "J5" H 3308 4420 50  0000 L CNN
+F 0 "J7" H 3308 4420 50  0000 L CNN
 F 1 "D-" H 3308 4329 50  0000 L CNN
 F 2 "RB-SMD-Connectors:TESTPOINT-1mm-NO_TEXT" H 3450 4300 50  0001 C CNN
@@
 	3250 4450 4550 4450
 $Comp
-L conn:TEST_1P J7
+L conn:TEST_1P J5
 U 1 1 5BAF56B7
 P 1650 4250
-F 0 "J7" H 1708 4370 50  0000 L CNN
+F 0 "J5" H 1708 4370 50  0000 L CNN
 F 1 "VBUS" H 1708 4279 50  0000 L CNN
 F 2 "RB-SMD-Connectors:TESTPOINT-1mm-NO_TEXT" H 1850 4250 50  0001 C CNN

Commit message: Adjustments to PCB
Changed lines of the file:
@@
 Text Label 9650 4650 0    60   ~ 0
 COL_12
+Text Label 9650 4450 0    60   ~ 0
+COL_10
 Text Label 9650 4550 0    60   ~ 0
-COL_10
-Text Label 9650 4450 0    60   ~ 0
 COL_11
 Text Label 9650 3550 0    60   ~ 0
@@
 Text Label 7150 3650 2    60   ~ 0
 COL_12
+Text Label 7150 3850 2    60   ~ 0
+COL_10
 Text Label 7150 3750 2    60   ~ 0
-COL_10
-Text Label 7150 3850 2    60   ~ 0
 COL_11
 Text Label 7150 5150 2    60   ~ 0

Commit message: Version 1.22 release
Small layout fix. ISP header changed to SMD test points.
Parts:
- J1, J2, J3, J4, J5, J6, J7, J8, J9: symbol conn:TEST_1P -> Keyboard-rescue:TEST_1P-conn
Changed lines of the file:
@@
 	9850 4850 9850 4950
 $Comp
-L conn:TEST_1P J6
+L Keyboard-rescue:TEST_1P-conn J6
 U 1 1 5BA336D5
 P 2700 4250
@@
 Connection ~ 2550 4350
 $Comp
-L conn:TEST_1P J9
+L Keyboard-rescue:TEST_1P-conn J9
 U 1 1 5BA4EE50
 P 1900 4800
@@
 Connection ~ 1650 4750
 $Comp
-L conn:TEST_1P J1
+L Keyboard-rescue:TEST_1P-conn J1
 U 1 1 5BA582A5
 P 6650 1000
@@
 $EndComp
 $Comp
-L conn:TEST_1P J3
+L Keyboard-rescue:TEST_1P-conn J3
 U 1 1 5BA6AA8B
 P 7350 1000
@@
 	7350 1300 8150 1300
 $Comp
-L conn:TEST_1P J2
+L Keyboard-rescue:TEST_1P-conn J2
 U 1 1 5BA74139
 P 7000 1000
@@
 	7000 1400 8150 1400
 $Comp
-L conn:TEST_1P J4
+L Keyboard-rescue:TEST_1P-conn J4
 U 1 1 5BABDEEC
 P 9450 1000
@@
 ICSP
 $Comp
-L conn:TEST_1P J8
+L Keyboard-rescue:TEST_1P-conn J8
 U 1 1 5BAC5EE6
 P 3250 4700
@@
 $EndComp
 $Comp
-L conn:TEST_1P J7
+L Keyboard-rescue:TEST_1P-conn J7
 U 1 1 5BAC5EEC
 P 3250 4300
@@
 	3250 4450 4550 4450
 $Comp
-L conn:TEST_1P J5
+L Keyboard-rescue:TEST_1P-conn J5
 U 1 1 5BAF56B7
 P 1650 4250
