File: TestRig/TestRig.sch (KiCad schematic (older format))
At the start: 17 parts, among them J1 USB_B_Micro, J2 AVR-ISP-6

Commit message: Should...
Parts:
- removed MH? (x4): MountingHole, MountingHole:MountingHole_3.2mm_M3, symbol Mechanical:MountingHole
- added A1: Arduino_UNO_R3, Module:Arduino_UNO_R3_WithMountingHoles, symbol MCU_Module:Arduino_UNO_R3
- added K1: PCB Jig 3D model, TestRig:PCB_JIG, symbol rbv_pcb_extras:DUMMY_KEY
- added K2: 3D Model Dummy, TestRig:USB_KEYBOARD_ADAPTER_V1.22_DUMMY, symbol rbv_pcb_extras:DUMMY_KEY
- added KB1: TO DUT, RB-SMD-Connectors:FPC_0.5mm_22p-MOLEX_52437, symbol rbv_keyboard:KEYBOARD-PSION-5MX
- added MH2: MountingHole, MountingHole:MountingHole_3.2mm_M3, symbol Mechanical:MountingHole
- TP1, TP2, TP3, TP4, TP5, TP6, TP7, TP8, TP9: footprint Connector_Pin:Pin_D1.0mm_L10.0mm -> RB-Connectors:Mill-Max_7911-0-15-20-86-14-11-0
- gave numbers to parts that had none: 2
Connections:
- net labels added: COL1, COL10, COL11, COL12, COL2, COL3, COL4, COL5, COL6, COL7, COL8, COL9, ROW1, ROW2, ROW3, ROW4, ROW5, ROW6, ROW7, ROW8
- wire segments 21 -> 67
- no-connect marks 1 -> 11
